File: dice.kicad_pcb (KiCad board)
At the start: 2 copper layers, 50 x 50 mm, 25 parts, among them P1 CONN_01X01, SW1 RUN, U1 74LS393, U2 74LS08, U3 74LS27, U4 74LS32, U5 555

Commit message: :cactus: :camel:
Parts:
- moved C1 11.9 mm to (81.9, 89.5)
- moved C2 11.9 mm to (89.4, 96.0)
- moved C3 11.9 mm to (94.4, 96.0)
- moved C4 11.9 mm to (86.4, 89.5)
- moved D1 11.9 mm to (73.9, 106.5)
- moved D2 11.9 mm to (91.9, 106.5)
- moved D3 11.9 mm to (73.9, 88.5)
- moved D4 11.9 mm to (108.9, 88.5)
- moved D5 11.9 mm to (108.9, 106.5)
- moved D6 11.9 mm to (108.9, 125.5)
- moved D7 11.9 mm to (73.9, 125.5)
- moved P1 11.9 mm to (81.9, 97.0)
- moved R1 11.9 mm to (102.9, 86.0)
- moved R2 11.9 mm to (102.4, 94.0)
- moved R3 11.9 mm to (110.4, 97.0)
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Routing:
- net GND: track 0.00 -> 21.7 mm, vias 0 -> 12
- net VCC: track 0.00 -> 7.92 mm, vias 0 -> 2
- net Net-(U1-Pad2): track 20.9 -> 20.1 mm, vias 0 -> 2
- net Net-(U1-Pad4): track 70.1 -> 69.4 mm, vias 4 -> 6
- net Net-(R1-Pad2): track 43.6 -> 43.7 mm, vias 0 -> 4
- net Net-(D4-Pad1): vias 1 -> 3
- added copper zone on B.Cu, net GND
- added copper zone on F.Cu, net VCC
Other:
- board text added: "5V"
- board text added: "LED Dice 2/22/16"
- board text added: "Tyler Spadgenske"

Commit message: v1 done :smile:
Parts:
- added P2: PWR, Socket_Strips:Socket_Strip_Straight_1x02, F.Cu at (70.3, 107.9)
- SW1: value RUN -> PWR
Routing:
- net GND: track 21.7 -> 26.5 mm, vias 12 -> 13
Changed lines of the file:
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@@
 (kicad_pcb (version 4) (host pcbnew 4.0.1-stable)
   (general
-    (links 51)
+    (links 53)
     (no_connects 0)
-    (area 75.124999 91.224999 125.275001 141.375001)
+    (area 64.075 79.775 118.175001 131.875001)
     (thickness 1.6)
     (drawings 7)
-    (tracks 244)
+    (tracks 248)
     (zones 0)
-    (modules 25)
+    (modules 26)
     (nets 24)
   )
@@
   (layers
     (0 F.Cu signal)
-    (31 B.Cu signal hide)
+    (31 B.Cu signal)
     (32 B.Adhes user)
     (33 F.Adhes user)
@@
     (visible_elements FFFFFF7F)
     (pcbplotparams
-      (layerselection 0x00030_80000001)
+      (layerselection 0x010f0_80000001)
       (usegerberextensions false)
       (excludeedgelayer true)
@@
       (outputformat 1)
       (mirror false)
-      (drillshape 1)
+      (drillshape 0)
       (scaleselection 1)
-      (outputdirectory ""))
+      (outputdirectory gerbers/))
   )
   (net 0 "")
@@
       (effects (font (size 1 1) (thickness 0.15)))
     )
-    (fp_text value RUN (at 1.2 4.2) (layer F.SilkS)
+    (fp_text value PWR (at 1.2 4.2) (layer F.SilkS)
       (effects (font (size 1 1) (thickness 0.15)))
     )
@@
       (scale (xyz 1 1 1))
       (rotate (xyz 0 0 90))
-    )
-  )
-  (module Socket_Strips:Socket_Strip_Straight_1x03 (layer F.Cu)
-    (at 90.4 84)
-    (descr "Through hole socket strip")
-    (tags "socket strip")
-    (fp_text reference SLOW (at -4.6 0) (layer F.SilkS)
-      (effects (font (size 1 1) (thickness 0.15)))
-    )
-    (fp_text value "SLOW PULSE" (at 0 -3.1) (layer F.Fab) hide
-      (effects (font (size 1 1) (thickness 0.15)))
-    )
-    (fp_line (start 0 -1.55) (end -1.55 -1.55) (layer F.SilkS) (width 0.15))
-    (fp_line (start -1.55 -1.55) (end -1.55 1.55) (layer F.SilkS) (width 0.15))
-    (fp_line (start -1.55 1.55) (end 0 1.55) (layer F.SilkS) (width 0.15))
-    (fp_line (start -1.75 -1.75) (end -1.75 1.75) (layer F.CrtYd) (width 0.05))
-    (fp_line (start 6.85 -1.75) (end 6.85 1.75) (layer F.CrtYd) (width 0.05))
-    (fp_line (start -1.75 -1.75) (end 6.85 -1.75) (layer F.CrtYd) (width 0.05))
-    (fp_line (start -1.75 1.75) (end 6.85 1.75) (layer F.CrtYd) (width 0.05))
-    (fp_line (start 1.27 -1.27) (end 6.35 -1.27) (layer F.SilkS) (width 0.15))
-    (fp_line (start 6.35 -1.27) (end 6.35 1.27) (layer F.SilkS) (width 0.15))
-    (fp_line (start 6.35 1.27) (end 1.27 1.27) (layer F.SilkS) (width 0.15))
-    (fp_line (start 1.27 1.27) (end 1.27 -1.27) (layer F.SilkS) (width 0.15))
-    (pad 1 thru_hole rect (at 0 0) (size 1.7272 2.032) (drill 1.016) (layers *.Cu *.Mask F.SilkS)
-      (net 2 GND))
-    (pad 2 thru_hole oval (at 2.54 0) (size 1.7272 2.032) (drill 1.016) (layers *.Cu *.Mask F.SilkS)
-      (net 5 "Net-(C4-Pad2)"))
-    (pad 3 thru_hole oval (at 5.08 0) (size 1.7272 2.032) (drill 1.016) (layers *.Cu *.Mask F.SilkS))
-    (model Socket_Strips.3dshapes/Socket_Strip_Straight_1x03.wrl
-      (at (xyz 0.1 0 0))
-      (scale (xyz 1 1 1))
-      (rotate (xyz 0 0 180))
     )
   )
@@
     )
   )
+  (module Socket_Strips:Socket_Strip_Straight_1x02 (layer F.Cu)
+    (at 70.3 107.9 90)
+    (descr "Through hole socket strip")
+    (tags "socket strip")
+    (fp_text reference P2 (at 0 -5.1 90) (layer F.SilkS) hide
+      (effects (font (size 1 1) (thickness 0.15)))
+    )
+    (fp_text value PWR (at -2.6 0.2 180) (layer F.SilkS)
+      (effects (font (size 1 1) (thickness 0.15)))
+    )
+    (fp_line (start -1.55 1.55) (end 0 1.55) (layer F.SilkS) (width 0.15))
+    (fp_line (start 3.81 1.27) (end 1.27 1.27) (layer F.SilkS) (width 0.15))
+    (fp_line (start -1.75 -1.75) (end -1.75 1.75) (layer F.CrtYd) (width 0.05))
+    (fp_line (start 4.3 -1.75) (end 4.3 1.75) (layer F.CrtYd) (width 0.05))
+    (fp_line (start -1.75 -1.75) (end 4.3 -1.75) (layer F.CrtYd) (width 0.05))
+    (fp_line (start -1.75 1.75) (end 4.3 1.75) (layer F.CrtYd) (width 0.05))
+    (fp_line (start 1.27 1.27) (end 1.27 -1.27) (layer F.SilkS) (width 0.15))
+    (fp_line (start 0 -1.55) (end -1.55 -1.55) (layer F.SilkS) (width 0.15))
+    (fp_line (start -1.55 -1.55) (end -1.55 1.55) (layer F.SilkS) (width 0.15))
+    (fp_line (start 1.27 -1.27) (end 3.81 -1.27) (layer F.SilkS) (width 0.15))
+    (fp_line (start 3.81 -1.27) (end 3.81 1.27) (layer F.SilkS) (width 0.15))
+    (pad 1 thru_hole rect (at 0 0 90) (size 2.032 2.032) (drill 1.016) (layers *.Cu *.Mask F.SilkS)
+      (net 1 VCC))
+    (pad 2 thru_hole oval (at 2.54 0 90) (size 2.032 2.032) (drill 1.016) (layers *.Cu *.Mask F.SilkS)
+      (net 2 GND))
+    (model Socket_Strips.3dshapes/Socket_Strip_Straight_1x02.wrl
+      (at (xyz 0.05 0 0))
+      (scale (xyz 1 1 1))
+      (rotate (xyz 0 0 180))
+    )
+  )
+  (module Socket_Strips:Socket_Strip_Straight_1x03 (layer F.Cu)
+    (at 90.4 84)
+    (descr "Through hole socket strip")
+    (tags "socket strip")
+    (fp_text reference SLOW (at -4.6 0.1) (layer F.SilkS)
+      (effects (font (size 1 1) (thickness 0.15)))
+    )
+    (fp_text value "SLOW PULSE" (at 0 -3.1) (layer F.Fab) hide
+      (effects (font (size 1 1) (thickness 0.15)))
+    )
+    (fp_line (start 0 -1.55) (end -1.55 -1.55) (layer F.SilkS) (width 0.15))
+    (fp_line (start -1.55 -1.55) (end -1.55 1.55) (layer F.SilkS) (width 0.15))
+    (fp_line (start -1.55 1.55) (end 0 1.55) (layer F.SilkS) (width 0.15))
+    (fp_line (start -1.75 -1.75) (end -1.75 1.75) (layer F.CrtYd) (width 0.05))
+    (fp_line (start 6.85 -1.75) (end 6.85 1.75) (layer F.CrtYd) (width 0.05))
+    (fp_line (start -1.75 -1.75) (end 6.85 -1.75) (layer F.CrtYd) (width 0.05))
+    (fp_line (start -1.75 1.75) (end 6.85 1.75) (layer F.CrtYd) (width 0.05))
+    (fp_line (start 1.27 -1.27) (end 6.35 -1.27) (layer F.SilkS) (width 0.15))
+    (fp_line (start 6.35 -1.27) (end 6.35 1.27) (layer F.SilkS) (width 0.15))
+    (fp_line (start 6.35 1.27) (end 1.27 1.27) (layer F.SilkS) (width 0.15))
+    (fp_line (start 1.27 1.27) (end 1.27 -1.27) (layer F.SilkS) (width 0.15))
+    (pad 1 thru_hole rect (at 0 0) (size 1.7272 2.032) (drill 1.016) (layers *.Cu *.Mask F.SilkS)
+      (net 2 GND))
+    (pad 2 thru_hole oval (at 2.54 0) (size 1.7272 2.032) (drill 1.016) (layers *.Cu *.Mask F.SilkS)
+      (net 5 "Net-(C4-Pad2)"))
+    (pad 3 thru_hole oval (at 5.08 0) (size 1.7272 2.032) (drill 1.016) (layers *.Cu *.Mask F.SilkS))
+    (model Socket_Strips.3dshapes/Socket_Strip_Straight_1x03.wrl
+      (at (xyz 0.1 0 0))
+      (scale (xyz 1 1 1))
+      (rotate (xyz 0 0 180))
+    )
+  )
   (gr_text 5V (at 91.8 106.2) (layer B.SilkS)
-    (effects (font (size 12.7 12.7) (thickness 0.3)))
+    (effects (font (size 12.7 12.7) (thickness 3)) (justify mirror))
   )
   (gr_text "LED\nDice\n2/22/16\n" (at 74.1 96.3) (layer F.SilkS)
@@
   (gr_line (start 68.1 131.8) (end 118.1 131.8) (angle 90) (layer Edge.Cuts) (width 0.15))
   (gr_line (start 68.1 81.8) (end 68.1 131.8) (angle 90) (layer Edge.Cuts) (width 0.15))
-  (segment (start 91.7 91.405) (end 93.695 91.405) (width 0.25) (layer F.Cu) (net 1) (status 400000))
-  (segment (start 95.905 87.595) (end 97.1 87.595) (width 0.25) (layer F.Cu) (net 1) (status 800000))
+  (segment (start 91.7 91.405) (end 93.695 91.405) (width 0.25) (layer F.Cu) (net 1))
+  (segment (start 95.905 87.595) (end 97.1 87.595) (width 0.25) (layer F.Cu) (net 1))
   (segment (start 94.8 88.7) (end 95.905 87.595) (width 0.25) (layer F.Cu) (net 1))
   (via (at 94.8 88.7) (size 0.6) (drill 0.4) (layers F.Cu B.Cu) (net 1))
@@
   (via (at 94 91.1) (size 0.6) (drill 0.4) (layers F.Cu B.Cu) (net 1))
   (segment (start 93.695 91.405) (end 94 91.1) (width 0.25) (layer F.Cu) (net 1))
+  (segment (start 70.3 105.36) (end 70.3 103.9) (width 0.25) (layer B.Cu) (net 2) (status 400000))
+  (segment (start 70.3 103.9) (end 69.6 103.2) (width 0.25) (layer B.Cu) (net 2))
+  (segment (start 90.4 84) (end 88.1 84) (width 0.25) (layer F.Cu) (net 2))
+  (via (at 88.1 84) (size 0.6) (drill 0.4) (layers F.Cu B.Cu) (net 2))
   (segment (start 91.7 87.595) (end 89.805 87.595) (width 0.25) (layer F.Cu) (net 2))
   (via (at 89.8 87.6) (size 0.6) (drill 0.4) (layers F.Cu B.Cu) (net 2))
@@
   (segment (start 96.4 97.5) (end 94.4 97.5) (width 0.25) (layer F.Cu) (net 4))
   (segment (start 99.9 94) (end 96.4 97.5) (width 0.25) (layer F.Cu) (net 4))
+  (segment (start 92.94 84) (end 92.94 84.96) (width 0.25) (layer F.Cu) (net 5))
+  (segment (start 92.94 84.96) (end 91.7 86.2) (width 0.25) (layer F.Cu) (net 5))
+  (segment (start 91.7 86.2) (end 88.2 86.2) (width 0.25) (layer F.Cu) (net 5))
+  (segment (start 88.2 86.2) (end 86.4 88) (width 0.25) (layer F.Cu) (net 5))
   (segment (start 86.4 88) (end 86.4 87.5) (width 0.25) (layer F.Cu) (net 5))
-  (segment (start 86.4 87.5) (end 87.9 86) (width 0.25) (layer F.Cu) (net 5))
-  (segment (start 87.9 86) (end 92.4 86) (width 0.25) (layer F.Cu) (net 5))
-  (segment (start 92.4 86) (end 92.94 85.46) (width 0.25) (layer F.Cu) (net 5))
-  (segment (start 92.94 85.46) (end 92.94 84) (width 0.25) (layer F.Cu) (net 5))
   (segment (start 111.44 106.5) (end 111.44 106.86) (width 0.25) (layer F.Cu) (net 6))
   (segment (start 111.44 106.86) (end 107.9 110.4) (width 0.25) (layer F.Cu) (net 6))
@@
   (segment (start 100.535 88.865) (end 97.1 88.865) (width 0.25) (layer F.Cu) (net 18))
   (segment (start 101.4 88) (end 100.535 88.865) (width 0.25) (layer F.Cu) (net 18))
-  (segment (start 104.4 86) (end 104.4 88.8) (width 0.25) (layer F.Cu) (net 19) (status 400000))
-  (segment (start 94.44 119.96) (end 94.44 125.5) (width 0.25) (layer F.Cu) (net 19) (status 800000))
+  (segment (start 104.4 86) (end 104.4 88.8) (width 0.25) (layer F.Cu) (net 19))
+  (segment (start 94.44 119.96) (end 94.44 125.5) (width 0.25) (layer F.Cu) (net 19))
   (segment (start 98.6 115.8) (end 94.44 119.96) (width 0.25) (layer F.Cu) (net 19))
   (via (at 98.6 115.8) (size 0.6) (drill 0.4) (layers F.Cu B.Cu) (net 19))
