File: dice.sch (KiCad schematic (older format))
At the start: 25 parts, among them P1 CONN_01X01, SW1 PWR, SW2 SLOW PULSE, U1 74LS393, U2 74LS08, U3 74LS27, U4 74LS32, U5 555

Commit message: :cactus: :camel:
Parts:
- added P2: PWR, symbol CONN_01X02
Connections:
- net GND: now also P2.2 (P2)
- net VCC: now also P2.1 (P1)
Changed lines of the file:
@@
 $EndComp
 $Comp
-L VCC #PWR01
+L VCC #PWR3
 U 1 1 56C8D637
 P 5000 1200
-F 0 "#PWR01" H 5000 1050 50  0001 C CNN
+F 0 "#PWR3" H 5000 1050 50  0001 C CNN
 F 1 "VCC" H 5000 1350 50  0000 C CNN
 F 2 "" H 5000 1200 60  0000 C CNN
@@
 $EndComp
 $Comp
-L VCC #PWR02
+L VCC #PWR1
 U 1 1 56C8DF7B
 P 4500 1750
-F 0 "#PWR02" H 4500 1600 50  0001 C CNN
+F 0 "#PWR1" H 4500 1600 50  0001 C CNN
 F 1 "VCC" H 4500 1900 50  0000 C CNN
 F 2 "" H 4500 1750 60  0000 C CNN
@@
 $EndComp
 $Comp
-L GND #PWR03
+L GND #PWR2
 U 1 1 56C8DFA5
 P 4500 2350
-F 0 "#PWR03" H 4500 2100 50  0001 C CNN
+F 0 "#PWR2" H 4500 2100 50  0001 C CNN
 F 1 "GND" H 4500 2200 50  0000 C CNN
 F 2 "" H 4500 2350 60  0000 C CNN
@@
 $EndComp
 $Comp
-L GND #PWR04
+L GND #PWR4
 U 1 1 56C8FB76
 P 5850 3300
-F 0 "#PWR04" H 5850 3050 50  0001 C CNN
+F 0 "#PWR4" H 5850 3050 50  0001 C CNN
 F 1 "GND" H 5850 3150 50  0000 C CNN
 F 2 "" H 5850 3300 60  0000 C CNN
@@
 $EndComp
 $Comp
-L GND #PWR05
+L GND #PWR7
 U 1 1 56C991CF
 P 9300 5200
-F 0 "#PWR05" H 9300 4950 50  0001 C CNN
+F 0 "#PWR7" H 9300 4950 50  0001 C CNN
 F 1 "GND" H 9300 5050 50  0000 C CNN
 F 2 "" H 9300 5200 60  0000 C CNN
@@
 Wire Wire Line
 	9300 4200 9300 5200
+$Comp
+L CONN_01X02 P2
+U 1 1 56CC0F10
+P 6950 3700
+F 0 "P2" H 6950 3850 50  0000 C CNN
+F 1 "PWR" H 7100 3700 50  0000 C CNN
+F 2 "" H 6950 3700 50  0000 C CNN
+F 3 "" H 6950 3700 50  0000 C CNN
+	1    6950 3700
+	1    0    0    -1
+$EndComp
+$Comp
+L VCC #PWR5
+U 1 1 56CC126D
+P 6650 3450
+F 0 "#PWR5" H 6650 3300 50  0001 C CNN
+F 1 "VCC" H 6650 3600 50  0000 C CNN
+F 2 "" H 6650 3450 50  0000 C CNN
+F 3 "" H 6650 3450 50  0000 C CNN
+	1    6650 3450
+	1    0    0    -1
+$EndComp
+$Comp
+L GND #PWR6
+U 1 1 56CC12B7
+P 6650 3950
+F 0 "#PWR6" H 6650 3700 50  0001 C CNN
+F 1 "GND" H 6650 3800 50  0000 C CNN
+F 2 "" H 6650 3950 50  0000 C CNN
+F 3 "" H 6650 3950 50  0000 C CNN
+	1    6650 3950
+	1    0    0    -1
+$EndComp
+Wire Wire Line
+	6750 3650 6650 3650
+Wire Wire Line
+	6650 3650 6650 3450
+Wire Wire Line
+	6750 3750 6650 3750
+Wire Wire Line
+	6650 3750 6650 3950
 $EndSCHEMATC

Commit message: v1 done :smile:
Parts:
- P2: footprint (none) -> Socket_Strips:Socket_Strip_Straight_1x02
Connections:
- net GND: no longer P2.2 (P2)
Changed lines of the file:
@@
 $EndComp
 $Comp
-L VCC #PWR3
+L VCC #PWR01
 U 1 1 56C8D637
 P 5000 1200
-F 0 "#PWR3" H 5000 1050 50  0001 C CNN
+F 0 "#PWR01" H 5000 1050 50  0001 C CNN
 F 1 "VCC" H 5000 1350 50  0000 C CNN
 F 2 "" H 5000 1200 60  0000 C CNN
@@
 $EndComp
 $Comp
-L VCC #PWR1
+L VCC #PWR02
 U 1 1 56C8DF7B
 P 4500 1750
-F 0 "#PWR1" H 4500 1600 50  0001 C CNN
+F 0 "#PWR02" H 4500 1600 50  0001 C CNN
 F 1 "VCC" H 4500 1900 50  0000 C CNN
 F 2 "" H 4500 1750 60  0000 C CNN
@@
 $EndComp
 $Comp
-L GND #PWR2
+L GND #PWR03
 U 1 1 56C8DFA5
 P 4500 2350
-F 0 "#PWR2" H 4500 2100 50  0001 C CNN
+F 0 "#PWR03" H 4500 2100 50  0001 C CNN
 F 1 "GND" H 4500 2200 50  0000 C CNN
 F 2 "" H 4500 2350 60  0000 C CNN
@@
 $EndComp
 $Comp
-L GND #PWR4
+L GND #PWR04
 U 1 1 56C8FB76
 P 5850 3300
-F 0 "#PWR4" H 5850 3050 50  0001 C CNN
+F 0 "#PWR04" H 5850 3050 50  0001 C CNN
 F 1 "GND" H 5850 3150 50  0000 C CNN
 F 2 "" H 5850 3300 60  0000 C CNN
@@
 $EndComp
 $Comp
-L GND #PWR7
+L GND #PWR05
 U 1 1 56C991CF
 P 9300 5200
-F 0 "#PWR7" H 9300 4950 50  0001 C CNN
+F 0 "#PWR05" H 9300 4950 50  0001 C CNN
 F 1 "GND" H 9300 5050 50  0000 C CNN
 F 2 "" H 9300 5200 60  0000 C CNN
@@
 	1    0    0    -1
 $EndComp
-Wire Wire Line
-	5000 1200 5000 2550
-Wire Wire Line
-	5000 1450 5050 1450
-Wire Wire Line
-	4500 1750 4500 1900
-Wire Wire Line
-	4500 2200 4500 2350
-Wire Wire Line
-	5650 1450 7100 1450
-Wire Wire Line
-	7100 1450 7100 1750
-Wire Wire Line
-	7100 2050 7100 2400
-Wire Wire Line
-	7100 2250 6600 2250
-Connection ~ 7100 2250
-Wire Wire Line
-	7100 2700 7100 3000
-Wire Wire Line
-	6600 2450 6950 2450
-Wire Wire Line
-	6650 2550 6650 2450
-Connection ~ 6650 2450
-Wire Wire Line
-	7100 2900 6950 2900
-Wire Wire Line
-	6950 2900 6950 2450
-Wire Wire Line
-	5200 2300 4850 2300
-Wire Wire Line
-	5200 2050 5100 2050
-Wire Wire Line
-	5100 2050 5100 1750
-Wire Wire Line
-	5100 1750 6700 1750
-Wire Wire Line
-	6700 1750 6700 2450
-Connection ~ 6700 2450
-Wire Wire Line
-	5000 2550 5200 2550
-Connection ~ 5000 1450
-Wire Wire Line
-	4850 2300 4850 2550
-Wire Wire Line
-	6650 3200 6650 2850
-Wire Wire Line
-	4850 2850 4850 3200
-Wire Wire Line
-	6600 2050 6750 2050
-Wire Wire Line
-	7100 3000 7050 3000
-Connection ~ 7100 2900
-Wire Wire Line
-	6750 3000 6250 3000
-Wire Wire Line
-	4850 3200 6650 3200
-Wire Wire Line
-	5850 3200 5850 3300
-Connection ~ 5850 3200
-Wire Wire Line
-	5250 3000 4850 3000
-Connection ~ 4850 3000
-Wire Wire Line
-	2550 4100 2400 4100
-Wire Wire Line
-	2300 4400 2550 4400
-Wire Wire Line
-	3950 4200 4250 4200
-Wire Wire Line
-	4250 4200 4250 5550
-Wire Wire Line
-	3950 4300 4150 4300
-Wire Wire Line
-	4150 4300 4150 4950
-Wire Wire Line
-	3950 4100 4550 4100
-Wire Wire Line
-	4250 4250 4550 4250
-Connection ~ 4250 4250
-Wire Wire Line
-	4550 4400 4150 4400
-Connection ~ 4150 4400
-Wire Wire Line
-	5750 4250 6450 4250
-Wire Wire Line
-	6000 4250 6000 4550
-Wire Wire Line
-	6000 4550 4450 4550
-Wire Wire Line
-	4450 4550 4450 4750
-Wire Wire Line
-	4450 4750 4550 4750
-Wire Wire Line
-	5750 4850 6450 4850
-Wire Wire Line
-	6000 4850 6000 5150
-Wire Wire Line
-	6000 5150 4450 5150
-Wire Wire Line
-	4450 5150 4450 5350
-Wire Wire Line
-	4450 5350 4550 5350
-Wire Wire Line
-	4250 5550 4550 5550
-Wire Wire Line
-	4150 4950 4550 4950
-Wire Wire Line
-	3950 4850 4150 4850
-Connection ~ 4150 4850
-Wire Wire Line
-	4250 5050 3950 5050
-Connection ~ 4250 5050
-Wire Wire Line
-	2750 4950 2300 4950
-Wire Wire Line
-	2300 4950 2300 4400
-Connection ~ 6000 4250
-Wire Wire Line
-	4350 3900 4200 3900
-Wire Wire Line
-	4200 3900 4200 4100
-Connection ~ 4200 4100
-Connection ~ 6000 4850
-Wire Wire Line
-	6450 5450 5750 5450
-Wire Wire Line
-	8300 4200 8050 4200
-Wire Wire Line
-	7650 4200 7400 4200
-Wire Wire Line
-	7400 4500 7650 4500
-Wire Wire Line
-	7400 4800 7650 4800
-Wire Wire Line
-	8050 4800 8300 4800
-Wire Wire Line
-	7400 5100 7650 5100
-Wire Wire Line
-	8050 5100 8300 5100
-Wire Wire Line
-	8700 4200 8850 4200
-Wire Wire Line
-	8700 4800 8850 4800
-Wire Wire Line
-	8700 5100 8850 5100
-Wire Wire Line
-	9150 4200 9300 4200
-Wire Wire Line
-	8050 4500 8850 4500
-Wire Wire Line
-	9150 4500 9300 4500
-Connection ~ 9300 4500
-Wire Wire Line
-	9300 4800 9150 4800
-Connection ~ 9300 4800
-Wire Wire Line
-	9300 5100 9150 5100
-Connection ~ 9300 5100
-Wire Wire Line
-	6750 1850 6650 1850
-Wire Wire Line
-	6650 1850 6650 2050
-Connection ~ 6650 2050
-Wire Wire Line
-	9300 4200 9300 5200
 $Comp
 L CONN_01X02 P2
@@
 F 0 "P2" H 6950 3850 50  0000 C CNN
 F 1 "PWR" H 7100 3700 50  0000 C CNN
-F 2 "" H 6950 3700 50  0000 C CNN
+F 2 "Socket_Strips:Socket_Strip_Straight_1x02" H 6950 3700 50  0001 C CNN
 F 3 "" H 6950 3700 50  0000 C CNN
 	1    6950 3700
@@
 $EndComp
 $Comp
-L VCC #PWR5
+L VCC #PWR06
 U 1 1 56CC126D
 P 6650 3450
-F 0 "#PWR5" H 6650 3300 50  0001 C CNN
+F 0 "#PWR06" H 6650 3300 50  0001 C CNN
 F 1 "VCC" H 6650 3600 50  0000 C CNN
 F 2 "" H 6650 3450 50  0000 C CNN
@@
 $EndComp
 $Comp
-L GND #PWR6
+L GND #PWR07
 U 1 1 56CC12B7
 P 6650 3950
-F 0 "#PWR6" H 6650 3700 50  0001 C CNN
+F 0 "#PWR07" H 6650 3700 50  0001 C CNN
 F 1 "GND" H 6650 3800 50  0000 C CNN
 F 2 "" H 6650 3950 50  0000 C CNN
@@
 $EndComp
 Wire Wire Line
+	5000 1200 5000 2550
+Wire Wire Line
+	5000 1450 5050 1450
+Wire Wire Line
+	4500 1750 4500 1900
+Wire Wire Line
+	4500 2200 4500 2350
+Wire Wire Line
+	5650 1450 7100 1450
+Wire Wire Line
+	7100 1450 7100 1750
+Wire Wire Line
+	7100 2050 7100 2400
+Wire Wire Line
+	7100 2250 6600 2250
+Connection ~ 7100 2250
+Wire Wire Line
+	7100 2700 7100 3000
+Wire Wire Line
+	6600 2450 6950 2450
+Wire Wire Line
+	6650 2550 6650 2450
+Connection ~ 6650 2450
+Wire Wire Line
+	7100 2900 6950 2900
+Wire Wire Line
+	6950 2900 6950 2450
+Wire Wire Line
+	5200 2300 4850 2300
+Wire Wire Line
+	5200 2050 5100 2050
+Wire Wire Line
+	5100 2050 5100 1750
+Wire Wire Line
+	5100 1750 6700 1750
+Wire Wire Line
+	6700 1750 6700 2450
+Connection ~ 6700 2450
+Wire Wire Line
+	5000 2550 5200 2550
+Connection ~ 5000 1450
+Wire Wire Line
+	4850 2300 4850 2550
+Wire Wire Line
+	6650 3200 6650 2850
+Wire Wire Line
+	4850 2850 4850 3200
+Wire Wire Line
+	6600 2050 6750 2050
+Wire Wire Line
+	7100 3000 7050 3000
+Connection ~ 7100 2900
+Wire Wire Line
+	6750 3000 6250 3000
+Wire Wire Line
+	4850 3200 6650 3200
+Wire Wire Line
+	5850 3200 5850 3300
+Connection ~ 5850 3200
+Wire Wire Line
+	5250 3000 4850 3000
+Connection ~ 4850 3000
+Wire Wire Line
+	2550 4100 2400 4100
+Wire Wire Line
+	2300 4400 2550 4400
+Wire Wire Line
+	3950 4200 4250 4200
+Wire Wire Line
+	4250 4200 4250 5550
+Wire Wire Line
+	3950 4300 4150 4300
+Wire Wire Line
+	4150 4300 4150 4950
+Wire Wire Line
+	3950 4100 4550 4100
+Wire Wire Line
+	4250 4250 4550 4250
+Connection ~ 4250 4250
+Wire Wire Line
+	4550 4400 4150 4400
+Connection ~ 4150 4400
+Wire Wire Line
+	5750 4250 6450 4250
+Wire Wire Line
+	6000 4250 6000 4550
+Wire Wire Line
+	6000 4550 4450 4550
+Wire Wire Line
+	4450 4550 4450 4750
+Wire Wire Line
+	4450 4750 4550 4750
+Wire Wire Line
+	5750 4850 6450 4850
+Wire Wire Line
+	6000 4850 6000 5150
+Wire Wire Line
+	6000 5150 4450 5150
+Wire Wire Line
+	4450 5150 4450 5350
+Wire Wire Line
+	4450 5350 4550 5350
+Wire Wire Line
+	4250 5550 4550 5550
+Wire Wire Line
+	4150 4950 4550 4950
+Wire Wire Line
+	3950 4850 4150 4850
+Connection ~ 4150 4850
+Wire Wire Line
+	4250 5050 3950 5050
+Connection ~ 4250 5050
+Wire Wire Line
+	2750 4950 2300 4950
+Wire Wire Line
+	2300 4950 2300 4400
+Connection ~ 6000 4250
+Wire Wire Line
+	4350 3900 4200 3900
+Wire Wire Line
+	4200 3900 4200 4100
+Connection ~ 4200 4100
+Connection ~ 6000 4850
+Wire Wire Line
+	6450 5450 5750 5450
+Wire Wire Line
+	8300 4200 8050 4200
+Wire Wire Line
+	7650 4200 7400 4200
+Wire Wire Line
+	7400 4500 7650 4500
+Wire Wire Line
+	7400 4800 7650 4800
+Wire Wire Line
+	8050 4800 8300 4800
+Wire Wire Line
+	7400 5100 7650 5100
+Wire Wire Line
+	8050 5100 8300 5100
+Wire Wire Line
+	8700 4200 8850 4200
+Wire Wire Line
+	8700 4800 8850 4800
+Wire Wire Line
+	8700 5100 8850 5100
+Wire Wire Line
+	9150 4200 9300 4200
+Wire Wire Line
+	8050 4500 8850 4500
+Wire Wire Line
+	9150 4500 9300 4500
+Connection ~ 9300 4500
+Wire Wire Line
+	9300 4800 9150 4800
+Connection ~ 9300 4800
+Wire Wire Line
+	9300 5100 9150 5100
+Connection ~ 9300 5100
+Wire Wire Line
+	6750 1850 6650 1850
+Wire Wire Line
+	6650 1850 6650 2050
+Connection ~ 6650 2050
+Wire Wire Line
+	9300 4200 9300 5200
+Wire Wire Line
 	6750 3650 6650 3650
 Wire Wire Line
 	6650 3650 6650 3450
-Wire Wire Line
-	6750 3750 6650 3750
-Wire Wire Line
-	6650 3750 6650 3950
 $EndSCHEMATC
